File: schematics/schmatics_desk_automation/_autosave-schmatics_desk_automation.kicad_pcb (KiCad board)
At the start: 2 copper layers, 122.5 x 110 mm, 12 parts, among them SW1 BT_UP, SW3 BT_DOWN, U1 L298N

Commit message: Add L298N interface library and enhance desk controller functionality
- Created a new symbol library for L298N interface in KiCad.
- Added autosave lock file for schematic design.
- Improved DeskController logic to handle error recovery from limit switches.
- Updated HAL initialization to set pin modes for upper and lower limit switches.
- Modified pin configuration for error LED and added definitions for limit switch inputs.
- Enhanced main loop to read limit switch states and integrate them into the application logic.
Parts:
- removed U1: L298N, DeskAutomation:L298N Interface
- added J1: L298N_Interface, DeskAutomation:L298N Interface, F.Cu at (163.8, 96.3)
- moved D3 21.9 mm to (170.0, 75.0)
- moved R_LED_DOWN1 21.9 mm to (169.5, 88.0)
- moved R_LED_ERROR_1 21.9 mm to (180.5, 83.0)
- moved R_LED_UP1 21.9 mm to (180.5, 87.0)
- moved D1 21.9 mm to (154.7, 75.4)
- moved D2 21.9 mm to (162.2, 75.4)
