File: schematics/schmatics_desk_automation/DeskAutomation_MotorControl/schmatics_no_arduino.kicad_sch (KiCad schematic)
At the start: 14 parts, among them J2 Conn_01x15_MountingPin, SW1 BT_UP, SW2 Lower Limit, SW3 BT_DOWN, SW4 Uppr Limit

Commit message: Remove autosave lock file for schematics desk automation
Parts:
- J2: footprint Connector_PinHeader_1.27mm:PinHeader_2x08_P1.27mm_Vertical -> (none)
- SW2, SW4: footprint SW_PUSH_6mm_H5mm -> (none)
Other:
- moved on the sheet: J2, L298N-Breakout1, R4, R5, R_LED_DOWN1, R_LED_ERROR_1, R_LED_UP1, SW1, SW2, SW3, SW4
